File: uClouds_002.brd (EAGLE design)
At the start: 40.6 x 128.5 mm, 147 parts, among them IC10 TL072D, IC11 74LS595D, IC2 LM1117-3.3, IC3 MCP6002, IC4 MCP6004, IC5 STM32F405RGT6, IC6 LM4040B10, IC7 LM1117-3.3, IC8 WM8731, IC9 TL072D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

Commit message: cleanup
Parts:
- moved BLEND 8.82 mm to (30.0, 88.4)
- moved C13 8.82 mm to (20.5, 94.4)
- moved C14 8.82 mm to (27.8, 33.5)
- moved C15 8.82 mm to (4.74, 46.5)
- moved C2 8.82 mm to (16.8, 73.5)
- moved C20 8.82 mm to (22.8, 50.5)
- moved C22 8.82 mm to (12.7, 44.1)
- moved C26 8.82 mm to (15.4, 59.4)
- moved C3 8.82 mm to (26.3, 64.3)
- moved IC11 8.82 mm to (33.2, 94.3)
- moved IC2 8.82 mm to (26.8, 74.6)
- moved IC6 8.82 mm to (22.1, 89.4)
- moved J2 8.82 mm to (19.8, 82.0)
- moved J3 8.82 mm to (5.85, 74.4)
- moved J6 8.82 mm to (33.8, 74.4)
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Other:
- board size 40.6 x 128.5 mm -> 39.6 x 110.9 mm
